File: hardware/ElevatorLift.kicad_sch (KiCad schematic)
At the start: 0 parts

Commit message: Capture portable Rev-A hardware design
Parts:
- added H1, H2, H3, H4: Mounting Hole 2.6mm, ElevatorLift_Custom:MountingHole_2.6mm_NPTH, symbol Mechanical:MountingHole
Other:
- added sheet Encoder_Counter (Encoder_Counter_RevA.kicad_sch)
- added sheet IO (IO.kicad_sch)
- added sheet MCU_Storage (MCU_Storage_RevA.kicad_sch)
- added sheet Power (Power_RevA.kicad_sch)
- added sheet VFD_Interface (VFD_Interface_RevA.kicad_sch)
