File: hardware/IO.kicad_sch (KiCad schematic)
At the start: 52 parts, among them J40 CONSMA002 (418 MHz ANT), J41 ED300/3 SAFETY HOME GND, J42 ED300/3 LIMIT UP DOWN GND, J43 ED300/3 SERVICE KEY HOLD GND, J44 ED300/3 SERVICE UP DOWN GND, J45 ED300/3 EXT LIGHT 12V / GND /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, J46 ED300/3 LIGHT + / SW- / GND, J47 ED300/3 AUX + / SW- / GND, Q40 AO3400A, Q41 AO3400A, SW40 RF LEARN, U40 RXM-418-LR, U41 LICAL-DEC-MS001, U42 TLP291-4, U43 TLP291-4

Commit message: Finalize Rev-A PCB preparation
Parts:
- removed D42: SMBJ15A, Diode_SMD:D_SMA, symbol Device:D_TVS
- removed F41: 500mA HOLD, Fuse:Fuse_1812_4532Metric, symbol Device:Polyfuse
- removed J47: ED300/3 AUX + / SW- / GND, TerminalBlock_Altech:Altech_AK300_1x03_P5.00mm_45-Degree, symbol Connector_Generic:Conn_01x03
- removed Q41: AO3400A, Package_TO_SOT_SMD:SOT-23, symbol Transistor_FET:AO3400A
- removed R59: 100R, Resistor_SMD:R_0603_1608Metric, symbol Device:R
- removed R60: 100k, Resistor_SMD:R_0603_1608Metric, symbol Device:R
- added R62: 1k, Resistor_SMD:R_0603_1608Metric, symbol Device:R
- R53: Reset_Strap (none) -> 10k to 3V3 biases GPIO3 HIGH with key open or 12V absent; c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
- TP40: footprint TestPoint:TestPoint_Plated_Hole_D2.0mm -> TestPoint:TestPoint_Pad_D1.0mm
Connections:
- net LIMIT_UP: now also R62.2; no longer R51.1, U42.12
- new net: R51.1, R62.1, U42.12
Other:
- note added: "OPTOCOUPLER-CONDITIONED 12 V FIELD INPUTS"
- note added: "Optional AUX output removed (R59/R60/Q41/F41/D42/J47). GPIO3 is now SERVICE_KEY, never an output. Field inputs remain active LOW (contact closed to GND). R62 limits GPIO43 ROM UART contention; validate startup."
- note removed: "ISOLATED 12 V FIELD INPUTS"
