File: hardware/MCU_Storage_RevA.kicad_sch (KiCad schematic)
At the start: 25 parts, among them J10 USB4145-03-0230-C_REVA2, J11 UART RECOVERY / BOOT, J12 RTC BACKUP 3V, SW10 RESET, SW11 BOOT, U10 ESP32-S3-WROOM-1U-N16R8, U11 PM004MNIATR 4Mbit MRAM, U12 TPD2EUSB30ADRTR USB ESD, U13 RV-3028-C7 RTC, U14 LM66100DCKR USB IDEAL DIODE

Commit message: Finalize Rev-A PCB preparation
Parts:
- J11: value UART RECOVERY / BOOT -> BOOT RESET HEADER - UART PINS 3/4 NC
- U10: Hardware_Contract (none) -> 2026-09-12: LIMIT_UP GPIO43/p37; LIMIT_DOWN GPIO44/p36; SER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
Connections:
- net AUX_CTRL is gone; now on net SERVICE_KEY: U10.15 (IO3)
- net LIMIT_DOWN: now also U10.36 (RXD0); no longer U10.29 (IO36)
- net LIMIT_UP: now also U10.37 (TXD0); no longer U10.28 (IO35)
- net SERVICE_KEY: no longer U10.30 (IO37)
- net UART0_RX: no longer names the net of J11.4 (Pin_4)
- net UART0_RX: no longer U10.36 (RXD0)
- net UART0_TX: no longer names the net of J11.3 (Pin_3)
- net UART0_TX: no longer U10.37 (TXD0)
- net VFD_ENABLE renamed VFD_COMMS_ENABLE
- no-connect marks 8 -> 13
Other:
- note added: "GPIO35/36/37: octal PSRAM, NC. GPIO43/44: limit inputs, no UART0 header. GPIO3 SERVICE_KEY: R53 10k pulls HIGH=open; LOW=closed. Keep default JTAG eFuses. Keep EFUSE_STRAP_JTAG_SEL=0; validate key states and supply sequencing during reset. Firmware: GPIO3/43/44 inputs, UART0 console disabled, GPIO42 UART OE only."
- note added: "U14 reverse-blocks USB VBUS into +5V. USB alone does NOT supply the 3V3 MCU rail. Use the approved isolated low-voltage bench supply procedure; do not assume USB-only operation."
- note removed: "U14 reverse-blocks USB VBUS before joining the regulated +5V rail, allowing safe USB programming with or without the AC/DC supply present."
Changed lines of the file:
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@@
 	(generator_version "10.0")
 	(paper "A3")
-	(text "ESP32-S3 native USB: GPIO19 = D-, GPIO20 = D+. U12 is the dedicated USB ESD array; CC1/CC2 each use 5.1k sink pull-downs."
+	(text "GPIO35/36/37: octal PSRAM, NC. GPIO43/44: limit inputs, no UART0 header.\nGPIO3 SERVICE_KEY: R53 10k pulls HIGH=open; LOW=closed. Keep default JTAG eFuses.\nKeep EFUSE_STRAP_JTAG_SEL=0; validate key states and supply sequencing during reset.\nFirmware: GPIO3/43/44 inputs, UART0 console disabled, GPIO42 UART OE only."
 		(exclude_from_sim no)
-		(at 35 170 0)
+		(at 160 185 0)
 		(effects
 			(font
-				(size 1 1)
+				(size 1.27 1.27)
 			)
 			(justify left bottom)
 		)
 	)
-	(text "U14 reverse-blocks USB VBUS before joining the regulated +5V rail, allowing safe USB programming with or without the AC/DC supply present."
+	(text "U14 reverse-blocks USB VBUS into +5V. USB alone does NOT supply the 3V3 MCU rail.\nUse the approved isolated low-voltage bench supply procedure; do not assume USB-only operation."
 		(exclude_from_sim no)
 		(at 80 58 0)
 		(effects
 			(font
+				(size 1.1 1.1)
+			)
+			(justify left bottom)
+		)
+	)
+	(text "ESP32-S3 native USB: GPIO19 = D-, GPIO20 = D+. U12 is the dedicated USB ESD array; CC1/CC2 each use 5.1k sink pull-downs."
+		(exclude_from_sim no)
+		(at 35 170 0)
+		(effects
+			(font
 				(size 1 1)
 			)
@@
 	)
 	(no_connect
+		(at 226.06 116.84)
+	)
+	(no_connect
+		(at 73.66 203.2)
+	)
+	(no_connect
+		(at 73.66 205.74)
+	)
+	(no_connect
 		(at 318.77 152.4)
 	)
@@
 	)
 	(no_connect
+		(at 226.06 119.38)
+	)
+	(no_connect
+		(at 226.06 114.3)
+	)
+	(no_connect
 		(at 125.73 86.36)
 	)
@@
 	(wire
 		(pts
+			(xy 308.61 143.51) (xy 306.07 144.78)
+		)
+		(stroke
+			(width 0)
+			(type default)
+		)
+	)
+	(wire
+		(pts
 			(xy 347.98 154.94) (xy 355.6 154.94)
 		)
@@
 		)
 	)
-	(label "UART0_TX"
-		(at 195.58 101.6 180)
-		(effects
-			(font
-				(size 1.27 1.27)
-			)
-			(justify right bottom)
-		)
-	)
 	(label "ESP_EN"
 		(at 167.64 88.9 180)
@@
 		)
 	)
-	(label "UART0_RX"
-		(at 73.66 203.2 0)
-		(effects
-			(font
-				(size 1.27 1.27)
-			)
-			(justify left bottom)
-		)
-	)
 	(label "ESP_BOOT"
 		(at 73.66 198.12 0)
@@
 		)
 	)
-	(label "UART0_RX"
-		(at 195.58 99.06 180)
-		(effects
-			(font
-				(size 1.27 1.27)
-			)
-			(justify right bottom)
-		)
-	)
 	(label "USB_VBUS_5V"
 		(at 43.18 99.06 180)
@@
 		)
 	)
-	(label "UART0_TX"
-		(at 73.66 205.74 0)
-		(effects
-			(font
-				(size 1.27 1.27)
-			)
-			(justify left bottom)
-		)
-	)
 	(label "USB_D-"
 		(at 78.74 106.68 0)
@@
 	)
 	(label "RTC_VBACKUP"
-		(at 306.07 144.78 90)
+		(at 308.61 143.51 90)
 		(effects
 			(font
@@
 		)
 	)
-	(global_label "SERVICE_KEY"
+	(global_label "LIMIT_UP"
 		(shape input)
-		(at 226.06 119.38 0)
+		(at 195.58 101.6 180)
 		(effects
 			(font
 				(size 1.27 1.27)
 			)
-			(justify left)
+			(justify right)
 		)
 		(property "Intersheetrefs" "${INTERSHEET_REFS}"
-			(at 226.06 119.38 0)
+			(at 195.58 101.6 0)
 			(hide yes)
 			(show_name no)
@@
 		)
 	)
-	(global_label "LIMIT_UP"
+	(global_label "RF_MODE_IND"
 		(shape input)
-		(at 226.06 114.3 0)
+		(at 226.06 99.06 0)
 		(effects
 			(font
@@
 		)
 		(property "Intersheetrefs" "${INTERSHEET_REFS}"
-			(at 226.06 114.3 0)
+			(at 226.06 99.06 0)
 			(hide yes)
 			(show_name no)
@@
 		)
 	)
-	(global_label "RF_MODE_IND"
+	(global_label "+5V"
 		(shape input)
-		(at 226.06 99.06 0)
+		(at 125.73 81.28 0)
 		(effects
 			(font
@@
 		)
 		(property "Intersheetrefs" "${INTERSHEET_REFS}"
-			(at 226.06 99.06 0)
+			(at 125.73 81.28 0)
 			(hide yes)
 			(show_name no)
@@
 		)
 	)
-	(global_label "+5V"
-		(shape input)
-		(at 125.73 81.28 0)
+	(global_label "SPI_MISO"
+		(shape output)
+		(at 322.58 99.02 0)
 		(effects
 			(font
@@
 		)
 		(property "Intersheetrefs" "${INTERSHEET_REFS}"
-			(at 125.73 81.28 0)
+			(at 322.58 99.02 0)
 			(hide yes)
 			(show_name no)
@@
 		)
 	)
-	(global_label "SPI_MISO"
-		(shape output)
-		(at 322.58 99.02 0)
+	(global_label "SERVICE_KEY"
+		(shape input)
+		(at 193.04 114.3 180)
 		(effects
 			(font
 				(size 1.27 1.27)
 			)
-			(justify left)
+			(justify right)
 		)
 		(property "Intersheetrefs" "${INTERSHEET_REFS}"
-			(at 322.58 99.02 0)
+			(at 193.04 114.3 0)
 			(hide yes)
 			(show_name no)
@@
 		)
 	)
-	(global_label "LIMIT_DOWN"
-		(shape input)
-		(at 226.06 116.84 0)
-		(effects
-			(font
-				(size 1.27 1.27)
-			)
-			(justify left)
-		)
-		(property "Intersheetrefs" "${INTERSHEET_REFS}"
-			(at 226.06 116.84 0)
-			(hide yes)
-			(show_name no)
-			(do_not_autoplace no)
-			(effects
-				(font
-					(size 1.27 1.27)
-				)
-			)
-		)
-	)
 	(global_label "HOME"
 		(shape input)
@@
 		)
 	)
-	(global_label "AUX_CTRL"
+	(global_label "SPI_MOSI"
 		(shape input)
-		(at 193.04 114.3 180)
+		(at 322.58 96.52 0)
 		(effects
 			(font
 				(size 1.27 1.27)
 			)
-			(justify right)
+			(justify left)
 		)
 		(property "Intersheetrefs" "${INTERSHEET_REFS}"
-			(at 193.04 114.3 0)
+			(at 322.58 96.52 0)
 			(hide yes)
 			(show_name no)
@@
 		)
 	)
-	(global_label "SPI_MOSI"
+	(global_label "VFD_COMMS_ENABLE"
 		(shape input)
-		(at 322.58 96.52 0)
+		(at 226.06 132.08 0)
 		(effects
 			(font
@@
 		)
 		(property "Intersheetrefs" "${INTERSHEET_REFS}"
-			(at 322.58 96.52 0)
+			(at 226.06 132.08 0)
 			(hide yes)
 			(show_name no)
@@
 		)
 	)
+	(global_label "LIMIT_DOWN"
+		(shape input)
+		(at 195.58 99.06 180)
+		(effects
+			(font
+				(size 1.27 1.27)
+			)
+			(justify right)
+		)
+		(property "Intersheetrefs" "${INTERSHEET_REFS}"
+			(at 195.58 99.06 0)
+			(hide yes)
+			(show_name no)
+			(do_not_autoplace no)
+			(effects
+				(font
+					(size 1.27 1.27)
+				)
+			)
+		)
+	)
 	(global_label "RF_D4"
 		(shape input)
@@
 		)
 	)
-	(global_label "VFD_ENABLE"
-		(shape output)
-		(at 226.06 132.08 0)
-		(effects
-			(font
-				(size 1.27 1.27)
-			)
-			(justify left)
-		)
-		(property "Intersheetrefs" "${INTERSHEET_REFS}"
-			(at 226.06 132.08 0)
-			(hide yes)
-			(show_name no)
-			(do_not_autoplace no)
-			(effects
-				(font
-					(size 1.27 1.27)
-				)
-			)
-		)
-	)
 	(global_label "SERVICE_UP"
 		(shape input)
@@
 			)
 		)
-		(property "Value" "UART RECOVERY / BOOT"
+		(property "Value" "BOOT RESET HEADER - UART PINS 3/4 NC"
 			(at 68.58 195.58 0)
 			(show_name no)
@@
 			)
 		)
+		(property "Hardware_Contract" "2026-09-12: LIMIT_UP GPIO43/p37; LIMIT_DOWN GPIO44/p36; SERVICE_KEY GPIO3/p15 active-low. GPIO35/36/37 reserved for octal PSRAM: NC. GPIO42 only VFD_COMMS_ENABLE. Native USB programming; UART0 disabled after boot. Keep default JTAG eFuses; SERVICE_KEY HIGH=open, LOW=closed; R53 10k pull-up."
+			(at 210.82 119.38 0)
+			(hide yes)
+			(show_name no)
+			(do_not_autoplace no)
+			(effects
+				(font
+					(size 1.27 1.27)
+				)
+			)
+		)
 		(pin "2"
 		)
@@
 		)
 		(property "Value" "RV-3028-C7 RTC"
-			(at 313.69 146.05 0)
+			(at 315.976 146.558 0)
 			(show_name no)
 			(do_not_autoplace no)
