File: hardware/Power_RevA.kicad_sch (KiCad schematic)
At the start: 24 parts, among them J20 Phoenix 1717732 GMKDS 1,5/3-7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, U20 AP63203WU 3V3 2A, U21 LM66100DCKR

Commit message: Finalize Rev-A PCB preparation
Parts:
- TP21, TP22: footprint TestPoint:TestPoint_Plated_Hole_D2.0mm -> TestPoint:TestPoint_Pad_D1.0mm
Changed lines of the file:
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@@
 			)
 		)
-		(property "Footprint" "TestPoint:TestPoint_Plated_Hole_D2.0mm"
+		(property "Footprint" "TestPoint:TestPoint_Pad_D1.0mm"
 			(at 255.27 172.72 0)
 			(hide yes)
@@
 			)
 		)
-		(property "Footprint" "TestPoint:TestPoint_Plated_Hole_D2.0mm"
+		(property "Footprint" "TestPoint:TestPoint_Pad_D1.0mm"
 			(at 224.79 113.03 0)
 			(hide yes)
