File: hardware/VFD_Interface_RevA.kicad_sch (KiCad schematic)
At the start: 11 parts, among them J24 VFD UART 5V GND RX TX, J25 ED300/3 VFD RUN C / E / SPARE, U24 TXS0104ED (3V3 <-> 5V), U25 VFD RUN OPEN COLLECTOR

Commit message: Finalize Rev-A PCB preparation
Parts:
- removed J25: ED300/3 VFD RUN C / E / SPARE, TerminalBlock_Altech:Altech_AK300_1x03_P5.00mm_45-Degree, symbol Connector_Generic:Conn_01x03
- removed R25: 680R, Resistor_SMD:R_0603_1608Metric, symbol Device:R
- removed TP26: VFD RUN COLLECTOR, TestPoint:TestPoint_Plated_Hole_D2.0mm, symbol Connector:TestPoint
- removed U25: VFD RUN OPEN COLLECTOR, Package_SO:SOIC-4_4.55x2.6mm_P1.27mm, symbol Isolator:TLP291
- TP24, TP25: footprint TestPoint:TestPoint_Plated_Hole_D2.0mm -> TestPoint:TestPoint_Pad_D1.0mm
- U24: Control_Authority (none) -> OE = GPIO42 VFD_COMMS_ENABLE only; R24 10k holds OE LOW at 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
Connections:
- net VFD_ENABLE renamed VFD_COMMS_ENABLE
- no-connect marks 5 -> 4
Other:
- note added: "COMMUNICATIONS ONLY - NO MCU RUN OUTPUT"
- note added: "OE = VFD_COMMS_ENABLE (GPIO42), default LOW via R24. UART mapping unchanged: ESP TX -> VFD RX; ESP RX <- VFD TX."
- note added: "R25/U25/J25/TP26 removed. Communications may operate with the safety chain open for STOP and readback. The separate external hardwired safety loop remains the sole RUN permission authority. Verify VFD configuration and wiring prohibit serial commands from bypassing the hardwired inhibit."
- note removed: "ISOLATED VFD RUN / ENABLE"
- note removed: "TXS0104E OE is pulled low and enabled only by VFD_ENABLE. UART mapping: ESP TX -> VFD RX; ESP RX <- VFD TX."
- note removed: "This RUN/ENABLE output is an operational stop path only. It is not a safety-rated circuit and does not replace the hardwired safety chain."
- note removed: "U25 presents an isolated open collector for a low-current VFD digital input. Verify VFD terminal voltage, polarity and required sink current before fitting J25."
